Commit message: feat:try bullet engine

File: assets/kuavo_s4/biped_s4.urdf (robot description, URDF)
Before this commit: robot biped_s4, 61 links, 60 joints
Links:
- link head_pitch: geometry collision mesh filename=package://meshes/head_pitch.STL; visual mesh filename=package://meshes/head_pitch.STL
- link head_yaw: geometry collision mesh filename=package://meshes/head_yaw.STL; visual mesh filename=package://meshes/head_yaw.STL
- link l_arm_pitch: geometry collision mesh filename=package://meshes/l_arm_pitch.STL; visual mesh filename=package://meshes/l_arm_pitch.STL
- link l_arm_roll: geometry collision mesh filename=package://meshes/l_arm_roll.STL; visual mesh filename=package://meshes/l_arm_roll.STL
- link l_arm_yaw: geometry collision mesh filename=package://meshes/l_arm_yaw.STL; visual mesh filename=package://meshes/l_arm_yaw.STL
- link l_foot_pitch: geometry collision mesh filename=package://meshes/l_foot_pitch.STL; visual mesh filename=package://meshes/l_foot_pitch.STL
- link l_foot_roll: geometry collision mesh filename=package://meshes/l_foot_roll.STL; visual mesh filename=package://meshes/l_foot_roll.STL
- link l_forearm_pitch: geometry collision mesh filename=package://meshes/l_forearm_pitch.STL; visual mesh filename=package://meshes/l_forearm_pitch.STL
- link l_hand_pitch: geometry collision mesh filename=package://meshes/l_hand_pitch.STL; visual mesh filename=package://meshes/l_hand_pitch.STL
- link l_hand_roll: geometry collision mesh filename=package://meshes/l_hand_roll.STL; visual mesh filename=package://meshes/l_hand_roll.STL
- link l_hand_yaw: geometry collision mesh filename=package://meshes/l_hand_yaw.STL; visual mesh filename=package://meshes/l_hand_yaw.STL
- link l_index_distal_finger: geometry collision mesh filename=package://meshes/l_index_distal_finger.STL; visual mesh filename=package://meshes/l_index_distal_finger.STL
- link l_index_proximal_finger: geometry collision mesh filename=package://meshes/l_index_proximal_finger.STL; visual mesh filename=package://meshes/l_index_proximal_finger.STL
- link l_knee: geometry collision mesh filename=package://meshes/l_knee.STL; visual mesh filename=package://meshes/l_knee.STL
- link l_l_bar: geometry collision mesh filename=package://meshes/l_l_bar.STL; visual mesh filename=package://meshes/l_l_bar.STL
- link l_l_tendon: geometry collision mesh filename=package://meshes/l_l_tendon.STL; visual mesh filename=package://meshes/l_l_tendon.STL
- link l_leg_pitch: geometry collision mesh filename=package://meshes/l_leg_pitch.STL; visual mesh filename=package://meshes/l_leg_pitch.STL
- link l_leg_roll: geometry collision mesh filename=package://meshes/l_leg_roll.STL; visual mesh filename=package://meshes/l_leg_roll.STL
- link l_leg_yaw: geometry collision mesh filename=package://meshes/l_leg_yaw.STL; visual mesh filename=package://meshes/l_leg_yaw.STL
- link l_middle_distal_finger: geometry collision mesh filename=package://meshes/l_middle_distal_finger.STL; visual mesh filename=package://meshes/l_middle_distal_finger.STL
- link l_middle_proximal_finger: geometry collision mesh filename=package://meshes/l_middle_proximal_finger.STL; visual mesh filename=package://meshes/l_middle_proximal_finger.STL
- link l_pinky_distal_finger: geometry collision mesh filename=package://meshes/l_pinky_distal_finger.STL; visual mesh filename=package://meshes/l_pinky_distal_finger.STL
- link l_pinky_proximal_finger: geometry collision mesh filename=package://meshes/l_pinky_proximal_finger.STL; visual mesh filename=package://meshes/l_pinky_proximal_finger.STL
- link l_r_bar: geometry collision mesh filename=package://meshes/l_r_bar.STL; visual mesh filename=package://meshes/l_r_bar.STL
- link l_r_tendon: geometry collision mesh filename=package://meshes/l_r_tendon.STL; visual mesh filename=package://meshes/l_r_tendon.STL
- link l_ring_distal_finger: geometry collision mesh filename=package://meshes/l_ring_distal_finger.STL; visual mesh filename=package://meshes/l_ring_distal_finger.STL
- link l_ring_proximal_finger: geometry collision mesh filename=package://meshes/l_ring_proximal_finger.STL; visual mesh filename=package://meshes/l_ring_proximal_finger.STL
- link l_thumb_distal_pitch: geometry collision mesh filename=package://meshes/l_thumb_distal_pitch.STL; visual mesh filename=package://meshes/l_thumb_distal_pitch.STL
- link l_thumb_proximal_yaw: geometry collision mesh filename=package://meshes/l_thumb_proximal_yaw.STL; visual mesh filename=package://meshes/l_thumb_proximal_yaw.STL
- link r_arm_pitch: geometry collision mesh filename=package://meshes/r_arm_pitch.STL; visual mesh filename=package://meshes/r_arm_pitch.STL
- link r_arm_roll: geometry collision mesh filename=package://meshes/r_arm_roll.STL; visual mesh filename=package://meshes/r_arm_roll.STL
- link r_arm_yaw: geometry collision mesh filename=package://meshes/r_arm_yaw.STL; visual mesh filename=package://meshes/r_arm_yaw.STL
- link r_foot_pitch: geometry collision mesh filename=package://meshes/r_foot_pitch.STL; visual mesh filename=package://meshes/r_foot_pitch.STL
- link r_foot_roll: geometry collision mesh filename=package://meshes/r_foot_roll.STL; visual mesh filename=package://meshes/r_foot_roll.STL
- link r_forearm_pitch: geometry collision mesh filename=package://meshes/r_forearm_pitch.STL; visual mesh filename=package://meshes/r_forearm_pitch.STL
- link r_hand_pitch: geometry collision mesh filename=package://meshes/r_hand_pitch.STL; visual mesh filename=package://meshes/r_hand_pitch.STL
- link r_hand_roll: geometry collision mesh filename=package://meshes/r_hand_roll.STL; visual mesh filename=package://meshes/r_hand_roll.STL
- link r_hand_yaw: geometry collision mesh filename=package://meshes/r_hand_yaw.STL; visual mesh filename=package://meshes/r_hand_yaw.STL
- link r_index_distal_finger: geometry collision mesh filename=package://meshes/r_index_distal_finger.STL; visual mesh filename=package://meshes/r_index_distal_finger.STL
- link r_index_proximal_finger: geometry collision mesh filename=package://meshes/r_index_proximal_finger.STL; visual mesh filename=package://meshes/r_index_proximal_finger.STL
- link r_knee: geometry collision mesh filename=package://meshes/r_knee.STL; visual mesh filename=package://meshes/r_knee.STL
- link r_l_bar: geometry collision mesh filename=package://meshes/r_l_bar.STL; visual mesh filename=package://meshes/r_l_bar.STL
- link r_l_tendon: geometry collision mesh filename=package://meshes/r_l_tendon.STL; visual mesh filename=package://meshes/r_l_tendon.STL
- link r_leg_pitch: geometry collision mesh filename=package://meshes/r_leg_pitch.STL; visual mesh filename=package://meshes/r_leg_pitch.STL
- link r_leg_roll: geometry collision mesh filename=package://meshes/r_leg_roll.STL; visual mesh filename=package://meshes/r_leg_roll.STL
- link r_leg_yaw: geometry collision mesh filename=package://meshes/r_leg_yaw.STL; visual mesh filename=package://meshes/r_leg_yaw.STL
- link r_middle_distal_finger: geometry collision mesh filename=package://meshes/r_middle_distal_finger.STL; visual mesh filename=package://meshes/r_middle_distal_finger.STL
- link r_middle_proximal_finger: geometry collision mesh filename=package://meshes/r_middle_proximal_finger.STL; visual mesh filename=package://meshes/r_middle_proximal_finger.STL
- link r_pinky_distal_finger: geometry collision mesh filename=package://meshes/r_pinky_distal_finger.STL; visual mesh filename=package://meshes/r_pinky_distal_finger.STL
- link r_pinky_proximal_finger: geometry collision mesh filename=package://meshes/r_pinky_proximal_finger.STL; visual mesh filename=package://meshes/r_pinky_proximal_finger.STL
- link r_r_bar: geometry collision mesh filename=package://meshes/r_r_bar.STL; visual mesh filename=package://meshes/r_r_bar.STL
- link r_r_tendon: geometry collision mesh filename=package://meshes/r_r_tendon.STL; visual mesh filename=package://meshes/r_r_tendon.STL
- link r_ring_distal_finger: geometry collision mesh filename=package://meshes/r_ring_distal_finger.STL; visual mesh filename=package://meshes/r_ring_distal_finger.STL
- link r_ring_proximal_finger: geometry collision mesh filename=package://meshes/r_ring_proximal_finger.STL; visual mesh filename=package://meshes/r_ring_proximal_finger.STL
- link r_thumb_distal_pitch: geometry collision mesh filename=package://meshes/r_thumb_distal_pitch.STL; visual mesh filename=package://meshes/r_thumb_distal_pitch.STL
- link r_thumb_proximal_yaw: geometry collision mesh filename=package://meshes/r_thumb_proximal_yaw.STL; visual mesh filename=package://meshes/r_thumb_proximal_yaw.STL
- link torso: geometry collision mesh filename=package://meshes/torso.STL; visual mesh filename=package://meshes/torso.STL

Commit message: fix:model file

File: assets/kuavo_s4/biped_s4.urdf (robot description, URDF)
Before this commit: robot biped_s4, 61 links, 60 joints
Joints:
- joint head_pitch: limit (none) -> lower=-3.14159 upper=3.14159 effort=20 velocity=1; type continuous -> revolute
- joint head_yaw: limit (none) -> lower=-3.14159 upper=3.14159 effort=20 velocity=1; type continuous -> revolute
- joint l_foot_pitch: limit (none) -> lower=-3.14159 upper=3.14159 effort=20 velocity=1; type continuous -> revolute
- joint l_foot_roll: limit (none) -> lower=-3.14159 upper=3.14159 effort=20 velocity=1; type continuous -> revolute
- joint l_index_distal_finger: limit (none) -> lower=-3.14159 upper=3.14159 effort=20 velocity=1; type continuous -> revolute
- joint l_index_proximal_finger: limit (none) -> lower=-3.14159 upper=3.14159 effort=20 velocity=1; type continuous -> revolute
- joint l_knee: limit (none) -> lower=-3.14159 upper=3.14159 effort=20 velocity=1; type continuous -> revolute
- joint l_l_bar: limit (none) -> lower=-3.14159 upper=3.14159 effort=20 velocity=1; type continuous -> revolute
- joint l_l_tendon: limit (none) -> lower=-3.14159 upper=3.14159 effort=20 velocity=1; type continuous -> revolute
- joint l_leg_pitch: limit (none) -> lower=-3.14159 upper=3.14159 effort=20 velocity=1; type continuous -> revolute
- joint l_leg_roll: limit (none) -> lower=-3.14159 upper=3.14159 effort=20 velocity=1; type continuous -> revolute
- joint l_leg_yaw: limit (none) -> lower=-3.14159 upper=3.14159 effort=20 velocity=1; type continuous -> revolute
- joint l_middle_distal_finger: limit (none) -> lower=-3.14159 upper=3.14159 effort=20 velocity=1; type continuous -> revolute
- joint l_middle_proximal_finger: limit (none) -> lower=-3.14159 upper=3.14159 effort=20 velocity=1; type continuous -> revolute
- joint l_pinky_distal_finger: limit (none) -> lower=-3.14159 upper=3.14159 effort=20 velocity=1; type continuous -> revolute
- joint l_pinky_proximal_finger: limit (none) -> lower=-3.14159 upper=3.14159 effort=20 velocity=1; type continuous -> revolute
- joint l_r_bar: limit (none) -> lower=-3.14159 upper=3.14159 effort=20 velocity=1; type continuous -> revolute
- joint l_r_tendon: limit (none) -> lower=-3.14159 upper=3.14159 effort=20 velocity=1; type continuous -> revolute
- joint l_ring_distal_finger: limit (none) -> lower=-3.14159 upper=3.14159 effort=20 velocity=1; type continuous -> revolute
- joint l_ring_proximal_finger: limit (none) -> lower=-3.14159 upper=3.14159 effort=20 velocity=1; type continuous -> revolute
- joint l_thumb_distal_pitch: limit (none) -> lower=-3.14159 upper=3.14159 effort=20 velocity=1; type continuous -> revolute
- joint l_thumb_proximal_yaw: limit (none) -> lower=-3.14159 upper=3.14159 effort=20 velocity=1; type continuous -> revolute
- joint r_foot_pitch: limit (none) -> lower=-3.14159 upper=3.14159 effort=20 velocity=1; type continuous -> revolute
- joint r_foot_roll: limit (none) -> lower=-3.14159 upper=3.14159 effort=20 velocity=1; type continuous -> revolute
- joint r_index_distal_finger: limit (none) -> lower=-3.14159 upper=3.14159 effort=20 velocity=1; type continuous -> revolute
- joint r_index_proximal_finger: limit (none) -> lower=-3.14159 upper=3.14159 effort=20 velocity=1; type continuous -> revolute
- joint r_knee: limit (none) -> lower=-3.14159 upper=3.14159 effort=20 velocity=1; type continuous -> revolute
- joint r_l_bar: limit (none) -> lower=-3.14159 upper=3.14159 effort=20 velocity=1; type continuous -> revolute
- joint r_l_tendon: limit (none) -> lower=-3.14159 upper=3.14159 effort=20 velocity=1; type continuous -> revolute
- joint r_leg_pitch: limit (none) -> lower=-3.14159 upper=3.14159 effort=20 velocity=1; type continuous -> revolute
- joint r_leg_roll: limit (none) -> lower=-3.14159 upper=3.14159 effort=20 velocity=1; type continuous -> revolute
- joint r_leg_yaw: limit (none) -> lower=-3.14159 upper=3.14159 effort=20 velocity=1; type continuous -> revolute
- joint r_middle_distal_finger: limit (none) -> lower=-3.14159 upper=3.14159 effort=20 velocity=1; type continuous -> revolute
- joint r_middle_proximal_finger: limit (none) -> lower=-3.14159 upper=3.14159 effort=20 velocity=1; type continuous -> revolute
- joint r_pinky_distal_finger: limit (none) -> lower=-3.14159 upper=3.14159 effort=20 velocity=1; type continuous -> revolute
- joint r_pinky_proximal_finger: limit (none) -> lower=-3.14159 upper=3.14159 effort=20 velocity=1; type continuous -> revolute
- joint r_r_bar: limit (none) -> lower=-3.14159 upper=3.14159 effort=20 velocity=1; type continuous -> revolute
- joint r_r_tendon: limit (none) -> lower=-3.14159 upper=3.14159 effort=20 velocity=1; type continuous -> revolute
- joint r_ring_distal_finger: limit (none) -> lower=-3.14159 upper=3.14159 effort=20 velocity=1; type continuous -> revolute
- joint r_ring_proximal_finger: limit (none) -> lower=-3.14159 upper=3.14159 effort=20 velocity=1; type continuous -> revolute
- joint r_thumb_distal_pitch: limit (none) -> lower=-3.14159 upper=3.14159 effort=20 velocity=1; type continuous -> revolute
- joint r_thumb_proximal_yaw: limit (none) -> lower=-3.14159 upper=3.14159 effort=20 velocity=1; type continuous -> revolute
